File: RoverWingBoard/RoverWing-V4.brd (EAGLE design)
At the start: 81.3 x 81.3 mm, 80 parts, among them J1 HEADER-VH, J10 HEADER-PH-4P, J11 HEADER-PH-3P, J12 HEADER-3X04, J13 HEADER-3X06", J14 HEADER-2X16, J15 HEADER-2X12, J16 DF13-4P-1.25DSA, J17 DF13-6P-1.25DSA, J2 HEADER-VH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

Commit message: minor updates
Parts:
- moved J11 0.38 mm to (20.8, 27.6)
Connections:
- net 5V: now also J11.2; no longer J11.3
- net GND: now also J11.3; no longer J11.2
Routing:
- net 5V: track 234.6 -> 235.6 mm
Other:
- board text added: "RoverWing V0.9 D. Bershadsky, A. Kirillov github.com/roverwing"
- board text removed: "RoverWing V0.4 D. Bershadsky, A. Kirillov github.com/roverwing"
Changed lines of the file:
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@@
 <?xml version="1.0" encoding="utf-8"?>
 <!DOCTYPE eagle SYSTEM "eagle.dtd">
-<eagle version="9.2.2">
+<eagle version="9.3.0">
 <drawing>
 <settings>
-<setting alwaysvectorfont="yes"/>
+<setting alwaysvectorfont="no"/>
 <setting keepoldvectorfont="yes"/>
 <setting verticaltext="up"/>
@@
 <text x="-29.9348" y="9.7418" size="0.889" layer="25" font="vector" ratio="15" rot="SR0">+</text>
 <text x="-34.6338" y="9.816196875" size="0.889" layer="25" font="vector" ratio="15" rot="SR0">-</text>
-<text x="33.274" y="-7.493" size="0.889" layer="25" font="vector" ratio="11" rot="R180">RoverWing V0.4
+<text x="33.274" y="-7.493" size="0.889" layer="25" font="vector" ratio="11" rot="R180">RoverWing V0.9
 D. Bershadsky, A. Kirillov
 github.com/roverwing</text>
@@
 <dimension x1="16.129" y1="37.719" x2="37.719" y2="16.129" x3="33.655" y3="33.655" textsize="1.778" layer="51"/>
 <dimension x1="37.719" y1="16.129" x2="27.051" y2="27.051" x3="36.88469375" y3="25.98505" textsize="1.778" layer="51"/>
-<text x="18.542" y="27.813" size="0.889" layer="25" font="vector" ratio="11" rot="SR45">GND</text>
-<text x="20.955" y="30.226" size="0.889" layer="25" font="vector" ratio="11" rot="SR45">5V</text>
+<text x="20.574" y="29.972" size="0.889" layer="25" font="vector" ratio="11" rot="SR45">GND</text>
+<text x="18.669" y="28.067" size="0.889" layer="25" font="vector" ratio="11" rot="SR45">5V</text>
 <text x="27.686" y="29.21" size="0.889" layer="25" font="vector" ratio="11" rot="SR135">NEOPIXEL</text>
 <text x="15.875" y="25.273" size="0.889" layer="25" font="vector" ratio="11" rot="SR45">DATA</text>
@@
 <attribute name="VALUE" x="39.37" y="-7.62" size="0.4064" layer="27" ratio="10" rot="R90"/>
 </element>
-<element name="J11" library="RoverWing" package="B3B-PH-K" value="HEADER-PH-3P" x="20.828" y="27.178" smashed="yes" rot="R225">
-<attribute name="PARTNO" value="B3B-PH-K-S(LF)(SN)" x="20.828" y="27.178" size="1.778" layer="27" rot="R225" display="off"/>
-<attribute name="VALUE" x="21.726025" y="30.7701" size="1.016" layer="27" ratio="10" rot="R225"/>
+<element name="J11" library="RoverWing" package="B3B-PH-K" value="HEADER-PH-3P" x="20.828" y="27.559" smashed="yes" rot="R225">
+<attribute name="PARTNO" value="B3B-PH-K-S(LF)(SN)" x="20.828" y="27.559" size="1.778" layer="27" rot="R225" display="off"/>
+<attribute name="VALUE" x="21.726025" y="31.1511" size="1.016" layer="27" ratio="10" rot="R225"/>
 </element>
 <element name="J8" library="RoverWing" package="B4B-PH-K" value="HEADER-PH-4P" x="29.64360625" y="-16.891" smashed="yes" rot="R135">
@@
 <wire x1="-1.512" y1="21.705" x2="-1.651" y2="21.844" width="0.254" layer="1"/>
 <wire x1="-1.651" y1="21.844" x2="-4.064" y2="21.844" width="0.254" layer="1"/>
-<contactref element="J11" pad="2"/>
-<via x="19.812" y="28.194" extent="1-16" drill="0.3937"/>
+<via x="22.352" y="30.607" extent="1-16" drill="0.3937"/>
+<contactref element="J11" pad="3"/>
 </signal>
 <signal name="3.3V">
@@
 <via x="-19.304" y="2.54" extent="1-16" drill="0.35"/>
 <via x="-15.24" y="-6.858" extent="1-16" drill="0.35"/>
-<wire x1="16.764" y1="32.766" x2="11.049" y2="38.481" width="1.524" layer="16"/>
+<wire x1="12.1285" y1="37.4015" x2="11.049" y2="38.481" width="1.524" layer="16"/>
 <wire x1="-15.24" y1="-6.858" x2="-16.637" y2="-6.858" width="0.254" layer="1"/>
 <wire x1="-16.637" y1="-6.858" x2="-21.844" y2="-12.065" width="0.254" layer="1"/>
@@
 <contactref element="J15" pad="6"/>
 <wire x1="-12.7" y1="-3.81" x2="-15.24" y2="-3.81" width="0.6096" layer="16"/>
-<contactref element="J11" pad="3"/>
 <wire x1="17.234740625" y1="22.27026875" x2="17.570471875" y2="22.606" width="0.254" layer="1"/>
 <wire x1="18.796" y1="22.606" x2="17.570471875" y2="22.606" width="0.254" layer="1"/>
-<via x="18.161" y="32.766" extent="1-16" drill="0.35"/>
+<via x="15.24" y="33.274" extent="1-16" drill="0.35"/>
 <wire x1="30.3507125" y1="-17.59810625" x2="24.366303125" y2="-23.582515625" width="0.4064" layer="16"/>
 <wire x1="24.366303125" y1="-23.582515625" x2="24.322725" y2="-23.582515625" width="0.4064" layer="16"/>
@@
 <wire x1="18.471696875" y1="-29.486140625" x2="16.2078375" y2="-31.75" width="0.4064" layer="16"/>
 <wire x1="16.2078375" y1="-31.75" x2="2.286" y2="-31.75" width="0.4064" layer="16"/>
-<wire x1="23.495" y1="24.903575" x2="25.47813125" y2="22.92044375" width="1.524" layer="16"/>
-<wire x1="22.2422125" y1="28.5922125" x2="23.495" y2="27.339425" width="1.524" layer="16"/>
-<wire x1="23.495" y1="27.339425" x2="23.495" y2="24.903575" width="1.524" layer="16"/>
-<wire x1="22.2422125" y1="28.5922125" x2="18.068425" y2="32.766" width="1.524" layer="16"/>
-<wire x1="18.068425" y1="32.766" x2="16.764" y2="32.766" width="1.524" layer="16"/>
-<wire x1="22.2422125" y1="28.5922125" x2="22.2422125" y2="26.0522125" width="0.254" layer="1"/>
-<wire x1="22.2422125" y1="26.0522125" x2="18.796" y2="22.606" width="0.254" layer="1"/>
-<wire x1="18.161" y1="32.766" x2="19.598971875" y2="34.203971875" width="0.254" layer="1"/>
+<wire x1="21.5265" y1="25.3365" x2="18.796" y2="22.606" width="0.254" layer="1"/>
 <wire x1="19.598971875" y1="34.203971875" x2="19.598971875" y2="34.330971875" width="0.254" layer="1"/>
-<wire x1="18.068425" y1="32.766" x2="18.161" y2="32.766" width="0" layer="19" extent="16-16"/>
+<contactref element="J11" pad="2"/>
+<wire x1="25.47813125" y1="22.92044375" x2="12.1285" y2="36.270075" width="1.524" layer="16"/>
+<wire x1="12.1285" y1="36.270075" x2="12.1285" y2="37.4015" width="1.524" layer="16"/>
+<wire x1="15.24" y1="33.274" x2="16.296971875" y2="34.330971875" width="0.254" layer="1"/>
+<wire x1="16.296971875" y1="34.330971875" x2="19.598971875" y2="34.330971875" width="0.254" layer="1"/>
+<wire x1="20.828" y1="27.559" x2="21.5265" y2="26.8605" width="0.254" layer="1"/>
+<wire x1="21.5265" y1="26.8605" x2="21.5265" y2="25.3365" width="0.254" layer="1"/>
+<wire x1="12.1285" y1="36.270075" x2="15.24" y2="33.274" width="0" layer="19" extent="16-16"/>
 <wire x1="2.286" y1="-31.623" x2="2.286" y2="-31.75" width="0" layer="19" extent="16-16"/>
 <wire x1="0.9144" y1="-30.2514" x2="1.0795" y2="-30.5435" width="0" layer="19" extent="1-16"/>
+<wire x1="21.5265" y1="25.3365" x2="25.47813125" y2="22.92044375" width="0" layer="19" extent="1-1"/>
 </signal>
 <signal name="SDA2">
@@
 <wire x1="16.59604375" y1="31.221084375" x2="16.59604375" y2="27.432" width="0.254" layer="1"/>
 <wire x1="16.59604375" y1="27.432" x2="16.59604375" y2="27.39104375" width="0.254" layer="1"/>
-<wire x1="19.413784375" y1="25.763784375" x2="17.74556875" y2="27.432" width="0.254" layer="1"/>
-<wire x1="17.74556875" y1="27.432" x2="16.59604375" y2="27.432" width="0.254" layer="1"/>
+<wire x1="19.413784375" y1="26.144784375" x2="18.12656875" y2="27.432" width="0.254" layer="1"/>
+<wire x1="18.12656875" y1="27.432" x2="16.59604375" y2="27.432" width="0.254" layer="1"/>
 </signal>
 <signal name="NEOPIXEL">
