File: RoverWingBoard/RoverWing-V095.sch (EAGLE design)
At the start: 80 parts, among them J1 HEADER-VH, J10 HEADER-PH-4P, J11 HEADER-PH-3P, J12 HEADER-3X04, J13 HEADER-3X06", J14 HEADER-2X16, J15 HEADER-2X12, J16 DF13-4P-1.25DSA, J17 DF13-6P-1.25DSA, J2 HEADER-VH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

Commit message: V095 - fixed NeoPixel signals and added the covers
Parts:
- removed R109: 1k, RoverWing:RES-SMD-0805
- added R12: 2.7k*4, RoverWing:RES_ARRAY-2.7KX40603X4
- R11: value 2.7k*4 -> 1k; device RoverWing:RES_ARRAY-2.7KX40603X4 -> RoverWing:RES-SMD-0805
Connections:
- net 3.3V: now also R12.1, R12.2, R12.3, R12.4; no longer R109.1, R11.2, R11.3, R11.4
- net SCL1: now also R12.8; no longer R11.8
- net SCL2: now also R12.5; no longer R11.5
- net SDA1: now also R12.7; no longer R11.7
- net SDA2: now also R12.6; no longer R11.6
- net SWCLK: now also R11.2; no longer R109.2
Changed lines of the file:
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@@
 <part name="GND14" library="RoverWing" deviceset="GND" device=""/>
 <part name="C1" library="RoverWing" deviceset="CAP-POL-SMD-8X10.5" device="" value="220uF"/>
-<part name="R109" library="RoverWing" deviceset="RES-SMD-0805" device="" value="1k"/>
-<part name="R11" library="RoverWing" deviceset="RES_ARRAY-2.7KX4" device="0603X4" value="2.7k*4"/>
+<part name="R11" library="RoverWing" deviceset="RES-SMD-0805" device="" value="1k"/>
+<part name="R12" library="RoverWing" deviceset="RES_ARRAY-2.7KX4" device="0603X4" value="2.7k*4"/>
 <part name="U$11" library="RoverWing" deviceset="FIDUCIAL" device=""/>
 <part name="U$13" library="RoverWing" deviceset="FIDUCIAL" device=""/>
@@
 <attribute name="VALUE" x="117.856" y="132.969" size="1.524" layer="96" ratio="10"/>
 </instance>
-<instance part="R109" gate="G$1" x="17.78" y="20.32" smashed="yes" rot="R90">
+<instance part="R11" gate="G$1" x="17.78" y="20.32" smashed="yes" rot="R90">
 <attribute name="NAME" x="16.51" y="16.51" size="1.524" layer="95" font="vector" ratio="10" rot="R90"/>
 <attribute name="VALUE" x="20.32" y="16.51" size="1.524" layer="95" font="vector" ratio="10" rot="R90"/>
 </instance>
-<instance part="R11" gate="G$1" x="104.14" y="22.86" smashed="yes">
+<instance part="R12" gate="G$1" x="104.14" y="22.86" smashed="yes">
 <attribute name="NAME" x="114.6556" y="30.7086" size="1.524" layer="95" ratio="10"/>
 <attribute name="VALUE" x="114.0206" y="28.1686" size="1.524" layer="95" ratio="10" rot="SR0"/>
@@
 <segment>
 <wire x1="17.78" y1="15.24" x2="17.78" y2="16.51" width="0.1524" layer="91"/>
-<pinref part="R109" gate="G$1" pin="1"/>
+<pinref part="R11" gate="G$1" pin="1"/>
 <label x="16.51" y="12.7" size="1.778" layer="95"/>
 </segment>
@@
 <wire x1="106.68" y1="7.62" x2="106.68" y2="12.7" width="0.1524" layer="91"/>
 <label x="106.68" y="27.94" size="1.778" layer="95" rot="R90"/>
-<pinref part="R11" gate="G$1" pin="1"/>
+<pinref part="R12" gate="G$1" pin="1"/>
 <wire x1="106.68" y1="12.7" x2="106.68" y2="17.78" width="0.1524" layer="91"/>
 <wire x1="106.68" y1="17.78" x2="106.68" y2="22.86" width="0.1524" layer="91"/>
 <wire x1="106.68" y1="22.86" x2="106.68" y2="30.48" width="0.1524" layer="91"/>
 <junction x="106.68" y="22.86"/>
-<pinref part="R11" gate="G$1" pin="2"/>
+<pinref part="R12" gate="G$1" pin="2"/>
 <junction x="106.68" y="17.78"/>
-<pinref part="R11" gate="G$1" pin="3"/>
+<pinref part="R12" gate="G$1" pin="3"/>
 <junction x="106.68" y="12.7"/>
-<pinref part="R11" gate="G$1" pin="4"/>
+<pinref part="R12" gate="G$1" pin="4"/>
 </segment>
 <segment>
@@
 <pinref part="TP2" gate="G$1" pin="TP"/>
 <wire x1="17.78" y1="24.13" x2="17.78" y2="30.48" width="0.1524" layer="91"/>
-<pinref part="R109" gate="G$1" pin="2"/>
+<pinref part="R11" gate="G$1" pin="2"/>
 </segment>
 <segment>
@@
 <wire x1="132.08" y1="22.86" x2="139.7" y2="22.86" width="0.1524" layer="91"/>
 <label x="134.62" y="22.86" size="1.778" layer="95"/>
-<pinref part="R11" gate="G$1" pin="8"/>
+<pinref part="R12" gate="G$1" pin="8"/>
 </segment>
 <segment>
@@
 <wire x1="132.08" y1="17.78" x2="139.7" y2="17.78" width="0.1524" layer="91"/>
 <label x="134.62" y="17.78" size="1.778" layer="95"/>
-<pinref part="R11" gate="G$1" pin="7"/>
+<pinref part="R12" gate="G$1" pin="7"/>
 </segment>
 <segment>
@@
 <wire x1="132.08" y1="12.7" x2="139.7" y2="12.7" width="0.1524" layer="91"/>
 <label x="134.62" y="12.7" size="1.778" layer="95"/>
-<pinref part="R11" gate="G$1" pin="6"/>
+<pinref part="R12" gate="G$1" pin="6"/>
 </segment>
 </net>
@@
 <wire x1="132.08" y1="7.62" x2="139.7" y2="7.62" width="0.1524" layer="91"/>
 <label x="134.62" y="7.62" size="1.778" layer="95"/>
-<pinref part="R11" gate="G$1" pin="5"/>
-</segment>
-</net>
+<pinref part="R12" gate="G$1" pin="5"/>
+</segment>
+</net>
