File: RoverWingBoard/RoverWing-V1.3.brd (EAGLE design)
At the start: 81.3 x 81.3 mm, 82 parts, among them J1 HEADER-VH, J10 HEADER-PH-4P, J11 HEADER-PH-3P, J12 HEADER-3X04, J13 HEADER-3X06", J14 HEADER-2X16, J15 HEADER-2X12, J16 DF13-4P-1.25DSA, J17 DF13-6P-1.25DSA, J2 HEADER-VH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

Commit message: version 1.4 of the board
Parts:
- R13, R14, R15, R16: value 2K -> 1.5K
Routing:
- net TX: track 31.2 -> 31.7 mm
