File: RoverWingBoard/RoverWing-V1.4.brd (EAGLE design)
At the start: 81.3 x 81.3 mm, 82 parts, among them CON1 XT30PW-M, J10 HEADER-PH-4P, J11 HEADER-PH-3P, J12 HEADER-3X04, J13 HEADER-3X06", J14 HEADER-2X16, J15 HEADER-2X12, J16 DF13-4P-1.25DSA, J17 DF13-6P-1.25DSA, J2 HEADER-VH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

Commit message: Update RoverWing-V1.4.brd
Routing:
- net GND: track 38.1 -> 39.9 mm, vias 75 -> 82
- added copper zone on layer 1, net SW
Changed lines of the file:
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@@
 </element>
 <element name="C2" library="RoverWing" package="0805" value="22uF" x="-16.51" y="-9.398" smashed="yes" rot="R180">
-<attribute name="NAME" x="-17.018" y="-11.176" size="0.889" layer="25" font="vector" ratio="11"/>
+<attribute name="NAME" x="-17.018" y="-11.684" size="0.889" layer="25" font="vector" ratio="11"/>
 <attribute name="VALUE" x="-14.605" y="-7.239" size="0.889" layer="27" ratio="11" rot="R180"/>
 </element>
@@
 </element>
 <element name="C4" library="RoverWing" package="0805" value="100nF" x="-23.622" y="0.762" smashed="yes">
-<attribute name="NAME" x="-24.257" y="1.778" size="0.889" layer="25" font="vector" ratio="11"/>
+<attribute name="NAME" x="-25.4" y="0" size="0.889" layer="25" font="vector" ratio="11" rot="R90"/>
 </element>
 <element name="C14" library="RoverWing" package="0805" value="100nF" x="-10.033" y="-25.654" smashed="yes" rot="R180">
@@
 </element>
 <element name="R1" library="RoverWing" package="0805" value="100k" x="-24.003" y="4.699" smashed="yes" rot="R180">
-<attribute name="NAME" x="-22.733" y="6.604" size="0.889" layer="25" font="vector" ratio="11" rot="R180"/>
+<attribute name="NAME" x="-23.876" y="3.683" size="0.889" layer="25" font="vector" ratio="11" rot="R180"/>
 </element>
 <element name="R2" library="RoverWing" package="0805" value="40.2k" x="-23.622" y="-4.699" smashed="yes">
-<attribute name="NAME" x="-25.4" y="-4.318" size="0.889" layer="25" font="vector" ratio="11" rot="R180"/>
+<attribute name="NAME" x="-26.162" y="-3.683" size="0.889" layer="25" font="vector" ratio="11" rot="R270"/>
 </element>
 <element name="R3" library="RoverWing" package="0805" value="5.49K" x="-23.622" y="-7.239" smashed="yes" rot="R180">
-<attribute name="NAME" x="-22.606" y="-5.334" size="0.889" layer="25" font="vector" ratio="11" rot="R180"/>
+<attribute name="NAME" x="-26.289" y="-6.096" size="0.889" layer="25" font="vector" ratio="11" rot="R270"/>
 </element>
 <element name="U2" library="RoverWing" package="SOT-23-8" value="MP2225" x="-18.542" y="-3.429" smashed="yes" rot="R90">
@@
 </element>
 <element name="C3" library="RoverWing" package="0805" value="100nF" x="-19.177" y="-6.5786" smashed="yes">
-<attribute name="NAME" x="-21.082" y="-7.8486" size="0.889" layer="25" font="vector" ratio="11" rot="R90"/>
+<attribute name="NAME" x="-18.1864" y="-7.747" size="0.889" layer="25" font="vector" ratio="11" rot="R180"/>
 </element>
 <element name="C5" library="RoverWing" package="0805" value="33pF" x="-23.622" y="-2.159" smashed="yes" rot="R180">
-<attribute name="NAME" x="-22.606" y="-3.175" size="0.889" layer="25" font="vector" ratio="11" rot="R180"/>
+<attribute name="NAME" x="-26.289" y="-1.397" size="0.889" layer="25" font="vector" ratio="11" rot="R270"/>
 </element>
 <element name="U3" library="RoverWing" package="SOT223" value="PMIC-AZ1117EH-3.3" x="4.953" y="-27.94" smashed="yes" rot="R270">
@@
 <attribute name="VALUE" x="0.684" y="21.35" size="0.4064" layer="27" rot="R180"/>
 </element>
-<element name="CON1" library="amass" package="XT30PW-M" value="XT30PW-M" x="-28.067" y="-1.397" smashed="yes" rot="R90">
-<attribute name="NAME" x="-24.257" y="-6.477" size="1.778" layer="25" rot="R90"/>
+<element name="CON1" library="amass" package="XT30PW-M" value="XT30PW-M" x="-28.067" y="-1.397" locked="yes" smashed="yes" rot="R90">
 <attribute name="VALUE" x="-41.567" y="-6.697" size="1.778" layer="27" rot="R90"/>
 </element>
@@
 <wire x1="-17.018" y1="-6.604" x2="-17.018" y2="-4.628" width="0.3048" layer="1"/>
 <wire x1="-17.018" y1="-4.628" x2="-17.242" y2="-4.404" width="0.3048" layer="1"/>
-<wire x1="-17.242" y1="-2.454" x2="-17.242" y2="-4.404" width="0" layer="19" extent="1-1"/>
+<via x="-20.066" y="-8.382" extent="1-16" drill="0.35"/>
+<wire x1="-20.066" y1="-6.5786" x2="-20.066" y2="-8.382" width="0.3048" layer="1"/>
+<via x="-20.828" y="1.778" extent="1-16" drill="0.35"/>
+<via x="-19.304" y="2.032" extent="1-16" drill="0.35"/>
+<via x="-28.448" y="3.556" extent="1-16" drill="0.35"/>
+<via x="-26.416" y="3.556" extent="1-16" drill="0.35"/>
+<via x="-26.416" y="2.54" extent="1-16" drill="0.35"/>
+<via x="-27.432" y="3.556" extent="1-16" drill="0.35"/>
+<wire x1="-26.416" y1="3.556" x2="-27.432" y2="3.556" width="0" layer="19" extent="1-1"/>
 </signal>
 <signal name="3.3V">
@@
 <vertex x="-34.308028125" y="6.7445875"/>
 <vertex x="-34.21768125" y="-6.523440625"/>
-<vertex x="-34.21768125" y="-6.523440625"/>
 <vertex x="-17.958984375" y="-22.680153125"/>
 <vertex x="-17.50785625" y="-22.71485625"/>
-<vertex x="-15.748" y="-20.955"/>
-<vertex x="-15.748" y="-20.701"/>
-<vertex x="-15.780771875" y="-20.668228125"/>
-<vertex x="-15.780771875" y="-20.033228125"/>
-<vertex x="-25.908" y="-3.065271875"/>
-<vertex x="-25.908" y="-3.065271875"/>
-<vertex x="-30.08871875" y="-0.222384375"/>
-<vertex x="-30.030834375" y="6.38881875"/>
+<vertex x="-15.494" y="-20.701"/>
+<vertex x="-15.494" y="-20.32"/>
+<vertex x="-19.037125" y="-16.370446875"/>
+<vertex x="-26.162" y="-9.245571875"/>
+<vertex x="-26.162" y="-2.892553125"/>
+<vertex x="-30.59260625" y="0.120259375"/>
+<vertex x="-30.54225625" y="5.87085625"/>
 <vertex x="-18.515709375" y="18.051153125"/>
 <vertex x="-18.50706875" y="19.251865625"/>
@@
 <via x="-19.05" y="18.288" extent="1-16" drill="0.3937"/>
 <contactref element="R5" pad="2"/>
-<via x="-31.623" y="6.985" extent="1-16" drill="0.35"/>
+<via x="-31.75" y="6.858" extent="1-16" drill="0.35"/>
 <contactref element="C19" pad="1"/>
 <contactref element="C20" pad="1"/>
@@
 <wire x1="-28.242" y1="9.271" x2="-29.337" y2="9.271" width="0.8128" layer="1"/>
 <wire x1="-29.337" y1="9.271" x2="-31.75" y2="6.858" width="0.8128" layer="1"/>
-<wire x1="-31.623" y1="6.985" x2="-31.75" y2="6.858" width="0" layer="19" extent="1-1"/>
 </signal>
 <signal name="N$14">
@@
 <contactref element="U6" pad="4"/>
 <contactref element="R8" pad="1"/>
-<wire x1="-14.245790625" y1="-14.9097375" x2="-12.8505" y2="-16.305028125" width="0.254" layer="1"/>
-<wire x1="-14.245790625" y1="-14.9097375" x2="-14.50020625" y2="-14.7118125" width="0" layer="19" extent="1-1"/>
+<wire x1="-14.50020625" y1="-14.7118125" x2="-12.906990625" y2="-16.305028125" width="0.3048" layer="1"/>
+<wire x1="-12.906990625" y1="-16.305028125" x2="-12.8505" y2="-16.305028125" width="0.3048" layer="1"/>
 </signal>
 <signal name="N$17">
@@
 <wire x1="-18.161" y1="0.273" x2="-22.244" y2="0.273" width="0.3048" layer="1"/>
 <wire x1="-22.244" y1="0.273" x2="-22.733" y2="0.762" width="0.3048" layer="1"/>
+<polygon width="0.0254" layer="1" thermals="no">
+<vertex x="-19.812" y="-0.508"/>
+<vertex x="-17.145" y="-0.508"/>
+<vertex x="-17.145" y="-1.27"/>
+<vertex x="-18.161" y="-2.286"/>
+<vertex x="-18.669" y="-2.286"/>
+<vertex x="-19.812" y="-1.143"/>
+</polygon>
 <wire x1="-18.161" y1="0.273" x2="-18.1102" y2="0.273" width="0" layer="19" extent="1-1"/>
 </signal>
@@
 <wire x1="-10.922" y1="-31.749" x2="-11.152" y2="-31.979" width="0.254" layer="1"/>
 </signal>
-<signal name="N$3">
-<via x="-20.066" y="-8.382" extent="1-16" drill="0.35"/>
+<signal name="N$6">
+<via x="-37.846" y="9.906" extent="1-16" drill="0.35"/>
+</signal>
+<signal name="N$8">
+<via x="-34.417" y="-20.193" extent="1-16" drill="0.35"/>
 </signal>
 </signals>

Commit message: Update RoverWing-V1.4.brd
Routing:
- net 5V: vias 16 -> 17
Changed lines of the file:
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@@
 <via x="-26.416" y="2.54" extent="1-16" drill="0.35"/>
 <via x="-27.432" y="3.556" extent="1-16" drill="0.35"/>
-<wire x1="-26.416" y1="3.556" x2="-27.432" y2="3.556" width="0" layer="19" extent="1-1"/>
 </signal>
 <signal name="3.3V">
@@
 <wire x1="-2.176" y1="19.8" x2="-3.798" y2="19.8" width="0.3048" layer="1"/>
 <wire x1="-3.798" y1="19.8" x2="-4.191" y2="20.193" width="0.3048" layer="1"/>
-<wire x1="-4.191" y1="20.193" x2="-5.969" y2="20.193" width="0.3048" layer="1"/>
+<wire x1="-4.191" y1="20.193" x2="-5.969" y2="20.193" width="0.508" layer="1"/>
 <wire x1="-5.969" y1="20.193" x2="-6.477" y2="20.193" width="0.3048" layer="1"/>
-<wire x1="-5.842" y1="22.225" x2="-5.842" y2="20.32" width="0.3048" layer="1"/>
+<wire x1="-5.842" y1="22.225" x2="-5.842" y2="20.32" width="0.508" layer="1"/>
 <wire x1="-5.842" y1="20.32" x2="-5.969" y2="20.193" width="0.3048" layer="1"/>
 <wire x1="-0.508" y1="23.622" x2="-0.508" y2="22.225" width="0.3048" layer="1"/>
@@
 <wire x1="-14.605" y1="33.909" x2="-10.033" y2="38.481" width="1.524" layer="16"/>
 <wire x1="-10.033" y1="38.481" x2="-4.064" y2="38.481" width="1.524" layer="16"/>
-<via x="-15.24" y="5.588" extent="1-16" drill="0.3937"/>
-<via x="-15.24" y="4.572" extent="1-16" drill="0.3937"/>
+<via x="-15.24" y="6.096" extent="1-16" drill="0.3937"/>
+<via x="-15.24" y="5.08" extent="1-16" drill="0.3937"/>
 <wire x1="-4.064" y1="38.481" x2="4.064" y2="38.481" width="1.524" layer="16"/>
 <wire x1="4.064" y1="38.481" x2="10.16" y2="38.481" width="1.524" layer="16"/>
@@
 <contactref element="J8" pad="3"/>
 <contactref element="R4" pad="2"/>
-<wire x1="-15.24" y1="-3.81" x2="-15.24" y2="3.556" width="1.524" layer="16"/>
-<wire x1="-15.24" y1="3.556" x2="-15.24" y2="23.622" width="1.524" layer="16"/>
+<wire x1="-15.24" y1="-3.81" x2="-15.24" y2="4.064" width="1.524" layer="16"/>
+<wire x1="-15.24" y1="4.064" x2="-15.24" y2="7.112" width="1.524" layer="16"/>
+<wire x1="-15.24" y1="7.112" x2="-15.24" y2="23.622" width="1.524" layer="16"/>
 <wire x1="-15.24" y1="23.622" x2="-14.605" y2="24.257" width="1.524" layer="16"/>
 <wire x1="-14.605" y1="24.257" x2="-14.605" y2="33.909" width="1.524" layer="16"/>
@@
 <vertex x="-14.730290625" y="2.921"/>
 </polygon>
-<via x="-15.24" y="3.556" extent="1-16" drill="0.35"/>
+<via x="-15.24" y="4.064" extent="1-16" drill="0.35"/>
 <polygon width="0.0254" layer="16" thermals="no">
 <vertex x="-14.732" y="2.921"/>
 <vertex x="-20.066" y="2.921"/>
 <vertex x="-20.447" y="3.302"/>
-<vertex x="-20.447" y="7.239"/>
-<vertex x="-19.685" y="8.001"/>
+<vertex x="-20.447" y="7.747"/>
+<vertex x="-20.193" y="8.001"/>
 <vertex x="-15.494" y="8.001"/>
 <vertex x="-14.732" y="7.239"/>
@@
 <wire x1="31.279196875" y1="17.373378125" x2="31.279196875" y2="14.861403125" width="0.508" layer="1"/>
 <wire x1="15.24" y1="28.194" x2="17.8435" y2="30.7975" width="0.508" layer="16"/>
-<wire x1="-22.987" y1="9.398" x2="-22.987" y2="7.239" width="0.3048" layer="1"/>
-<wire x1="-20.193" y1="7.239" x2="-19.812" y2="7.62" width="0.3048" layer="1"/>
-<wire x1="-22.987" y1="7.239" x2="-20.193" y2="7.239" width="0.3048" layer="1"/>
+<wire x1="-22.987" y1="9.398" x2="-22.987" y2="7.239" width="0.508" layer="1"/>
+<wire x1="-20.193" y1="7.239" x2="-19.812" y2="7.62" width="0.508" layer="1"/>
+<wire x1="-22.987" y1="7.239" x2="-20.193" y2="7.239" width="0.508" layer="1"/>
 <wire x1="-15.24" y1="-11.43" x2="-22.225" y2="-11.43" width="0.3048" layer="16"/>
 <wire x1="-22.225" y1="-11.43" x2="-22.352" y2="-11.43" width="0.3048" layer="16"/>
@@
 <wire x1="-22.225" y1="-11.43" x2="-22.257" y2="-11.398" width="0.3048" layer="1"/>
 <wire x1="-22.257" y1="-11.398" x2="-27.619" y2="-11.398" width="0.3048" layer="1"/>
+<via x="-15.24" y="7.112" extent="1-16" drill="0.35"/>
 <wire x1="2.286" y1="-31.75" x2="2.286" y2="-31.623" width="0" layer="19" extent="16-16"/>
 <wire x1="0.9144" y1="-30.2514" x2="1.0795" y2="-30.5435" width="0" layer="19" extent="1-16"/>
@@
 <contactref element="C4" pad="2"/>
 <wire x1="-17.242" y1="-3.104" x2="-18.232" y2="-3.104" width="0.3048" layer="1"/>
-<wire x1="-18.232" y1="-3.104" x2="-18.415" y2="-2.921" width="0.3048" layer="1"/>
+<wire x1="-18.232" y1="-3.104" x2="-18.415" y2="-2.921" width="0.508" layer="1"/>
 <wire x1="-18.1102" y1="0.0561375" x2="-18.1102" y2="0.273" width="0.3048" layer="1"/>
-<wire x1="-18.415" y1="-2.921" x2="-18.415" y2="-0.2486625" width="0.3048" layer="1"/>
+<wire x1="-18.415" y1="-2.921" x2="-18.415" y2="-0.2486625" width="0.508" layer="1"/>
 <wire x1="-18.415" y1="-0.2486625" x2="-18.1102" y2="0.0561375" width="0.3048" layer="1"/>
 <wire x1="-18.161" y1="0.273" x2="-22.244" y2="0.273" width="0.3048" layer="1"/>
