File: Extras/RoverWing-cover-V1.5.brd (EAGLE design)
At the start: 81.3 x 81.3 mm, 52 parts, among them J1 HEADER-PH-3PSIDEENTRY, J10 HEADER-PH-6PSIDEENTRY, J13 HEADER-PH-6PSIDEENTRY, J16 FEATHERWING_NODIM, J17 HEADER-PH-6PSIDEENTRY, J5 HEADER-PH-6PSIDEENTRY

Commit message: docs update
Parts:
- moved J1 4.67 mm to (21.4, 27.7)
- moved J2 2.54 mm to (17.8, 19.1)
- moved S1 1.37 mm to (-10.2, -30.5)
Routing:
- net GND: track 168.9 -> 188.8 mm
- net 5V: track 134.3 -> 139.4 mm
- net NEOPIXEL_OUT: track 18.3 -> 23.0 mm
- net SCL: track 34.1 -> 37.7 mm
- net 3.3V: track 58.0 -> 60.5 mm
- net FEATHER_RESET: track 36.0 -> 34.9 mm
Other:
- outline, holes or cut-outs redrawn
