File: Extras/RoverWing-cover-V1.5.sch (EAGLE design)
At the start: 52 parts, among them J1 HEADER-PH-3PSIDEENTRY, J10 HEADER-PH-6PSIDEENTRY, J13 HEADER-PH-6PSIDEENTRY, J16 FEATHERWING_NODIM, J17 HEADER-PH-6PSIDEENTRY, J5 HEADER-PH-6PSIDEENTRY

Commit message: docs update
Other:
- moved on the sheet: C1, C2, C3, J16, J3, J4, S1, S2, S3
