File: Extras/RoverWing-cover-V2.0.sch (EAGLE design)
At the start: 52 parts, among them J1 HEADER-PH-3PSIDEENTRY, J10 HEADER-PH-6PSIDEENTRY, J13 HEADER-PH-6PSIDEENTRY, J16 FEATHERWING_NODIM, J17 HEADER-PH-6PSIDEENTRY, J5 HEADER-PH-6PSIDEENTRY

Commit message: asd
asd
Parts:
- C1, C2, C3: MF (none) -> AVX; MPN (none) -> 04025C104KAT2A; OC_NEWARK (none) -> 96Y8186
- FRAME2, J10, J101, J102, J103, J104, J105, J106, J107, J108, J109, J11, J110, J111, J112, J113, J114, J115, J116, J117, J12, J13, J14, J15, J16, J17, J2, J3, J4, J5, J6, J7, J8, J9, U$14, U$15, U$24, U$25, U$26, U$27, U$3, U$4: OC_NEWARK (none) -> unknown
- J1: MF (none) -> JST (JAPAN SOLDERLESS TERMINALS); MPN (none) -> S3B-PH-K-S (LF)(SN); OC_NEWARK (none) -> 38K8070
- LED1, LED2, LED3: MF (none) -> ADAFRUIT; MPN (none) -> 2659; OC_NEWARK (none) -> 77Y5297
- S1, S2, S3: MF (none) -> E-SWITCH; MPN (none) -> TL3305AF160QG; OC_NEWARK (none) -> 84Y2774
