File: RoverWingBoard/Eagle/RoverWing-V1.5.brd (EAGLE design)
At the start: 81.3 x 81.3 mm, 83 parts, among them J1 HEADER-VH, J10 HEADER-PH-4P, J11 HEADER-PH-3P, J12 HEADER-3X04, J13 HEADER-3X06", J14 HEADER-2X16, J15 HEADER-2X12, J16 DF13-4P-1.25DSA, J17 DF13-6P-1.25DSA, J2 HEADER-VH, J3 HEADER-VH, J4 HEADER-PH-4P, J5 HEADER-PH-4P, J6 HEADER-PH-4P, J8 HEADER-PH-4P, J9 HEADER-PH-4P, SW1 SW-TACTILE-4.5X4.5_SMD, U1 ATSAMD21G, U2 MP2225, U3 PMIC-AZ1117EH-3.3, U4 MPU-6050, U5 DRV8871, U6 DRV8871, U7 TXS0104EPWR, U8 74AHCT1G125DBV

Commit message: docs update
Parts:
- removed C16: 100nF, RoverWing:0805
- removed U4: MPU-6050, RoverWing:QFN50P400X400X95-24N
- added U9: ICM-42605, RoverWing-V1.5:PQFN50P300X250X97-14N
- C1: device RoverWing:CAP-8X10.5 -> RoverWing-V1.5:CAP-8X10.5
- C10, C11, C12, C13, C14, C15, C17, C18, C19, C2, C20, C3, C4, C5, C6, C7, C8, C9, FB, R1, R10, R11, R2, R3, R4, R5, R6, R7, R8: device RoverWing:0805 -> RoverWing-V1.5:0805
- C21: device RoverWing:CAP-6.3X5.4 -> RoverWing-V1.5:CAP-8X10.5
- D1: device RoverWing:LED-0805 -> RoverWing-V1.5:LED-0805
- D2: device RoverWing:LED3535 -> RoverWing-V1.5:LED3535
- FRAME1, FRAME2: device RoverWing:DUMMY -> RoverWing-V1.5:DUMMY
- J1: value HEADER-VH -> XT30UPB-M; device RoverWing:B2P-VH -> RoverWing-V1.5:XT30UPB-M
- J10, J4, J5, J6, J8, J9: device RoverWing:B4B-PH-K -> RoverWing-V1.5:B4B-PH-K
- J11: device RoverWing:B3B-PH-K -> RoverWing-V1.5:B3B-PH-K
- J12: device RoverWing:3X04 -> RoverWing-V1.5:3X04
- J13: device RoverWing:3X06 -> RoverWing-V1.5:3X06
- J14: device RoverWing:2X16 -> RoverWing-V1.5:2X16
- J15: device RoverWing:2X12 -> RoverWing-V1.5:2X12
- J16: device RoverWing:DF13-4P-1.25DSA -> RoverWing-V1.5:DF13-4P-1.25DSA
- J17: device RoverWing:DF13-6P-1.25DSA -> RoverWing-V1.5:DF13-6P-1.25DSA
- J2, J3: device RoverWing:B2P-VH -> RoverWing-V1.5:B2P-VH
- L1: device RoverWing:IND_TDK_7.1X6.5 -> RoverWing-V1.5:IND_TDK_7.1X6.5
- R13, R14, R15, R16: value 2K -> 1.8K; device Seeed-Resistor:R0603 -> RoverWing-V1.5:R0603
- SW1: device RoverWing:TL3305 -> RoverWing-V1.5:TL3305
- TP1, TP2, TP3, TP4, TP5: device RoverWing:TP15R -> RoverWing-V1.5:TP15R
- U$11, U$13, U$17: device RoverWing:FIDUCIAL_1MM -> RoverWing-V1.5:FIDUCIAL_1MM
- U$14, U$15, U$24, U$25, U$26, U$27, U$3, U$4: device RoverWing:MOUNTINGHOLE_3.0_NPH -> RoverWing-V1.5:MOUNTINGHOLE_3.0_NPH
- U1: device RoverWing:TQFP-48-EDITED -> RoverWing-V1.5:TQFP-48-EDITED
- U2: device RoverWing:SOT-23-8 -> RoverWing-V1.5:SOT-23-8
- U3: device RoverWing:SOT223 -> RoverWing-V1.5:SOT223
- U5, U6: device RoverWing:HSOP8 -> RoverWing-V1.5:HSOP8
- U7: device RoverWing:PW14 -> RoverWing-V1.5:PW14
- U8: device RoverWing:SOT23-5 -> RoverWing-V1.5:SOT23-5
- USB1: device RoverWing:MICRO-USB5+6P-SMD-0.65-B -> RoverWing-V1.5:MICRO-USB5+6P-SMD-0.65-B
- moved C21 7.55 mm to (23.9, 10.9), turned to 0 degrees
- moved C15 5.82 mm to (-6.48, 19.3), turned to 90 degrees
- moved C17 5.00 mm to (-4.19, 19.3), turned to 90 degrees
- moved C1 4.50 mm to (-35.4, 7.62)
- moved J1 4.31 mm to (-37.1, -4.57)
- moved J3 2.92 mm to (-22.0, -28.4), turned to 135 degrees
- moved J2 2.50 mm to (-28.3, 22.0), turned to 45 degrees
- moved D1 1.40 mm to (-32.5, -12.2)
- moved C18 0.51 mm to (-0.51, 24.5), turned to 90 degrees
Connections:
- net N$25 renamed NEOPIXEL_INTERNAL
- removed net N$4: J2.2, U5.8
- removed net N$6: C15.2, U4.10
- net 12V: now also J1.+; no longer J1.2
- net 3.3V: now also C15.2, C17.2, C18.1, U9.12, U9.5, U9.8; no longer C16.2, C18.2, U4.13, U4.8, U4.9
- net GND: now also C18.2, J1.-, U9.1, U9.6, U9.7, U9.9; no longer C16.1, C18.1, J1.1, U4.1, U4.11, U4.18
- net N$1: now also J3.1; no longer J3.2
- net N$16: now also J2.2; no longer J2.1
- net N$2: now also J3.2; no longer J3.1
- net N$3: now also J2.1, U5.8; no longer C17.2, U4.20
- net SCL2: now also U9.13; no longer U4.23
- net SDA2: now also U9.14; no longer U4.24
Routing:
- net 5V: track 238.1 -> 248.7 mm
- net 3.3V: track 261.9 -> 270.2 mm, vias 12 -> 13
- net N$3: track 2.32 -> 9.69 mm
- net GND: track 50.0 -> 43.6 mm, vias 101 -> 94
- net N$4: track 6.30 -> 0.00 mm
- net N$1: track 6.72 -> 10.1 mm
- net 12V: track 14.8 -> 18.2 mm, vias 14 -> 16
- net N$6: track 3.29 -> 0.00 mm
- net N$2: track 6.65 -> 9.74 mm
- net N$16: track 6.53 -> 9.15 mm
- net SDA2: track 35.8 -> 37.4 mm
- net N$17: track 6.99 -> 5.64 mm
- net SCL2: track 34.1 -> 35.4 mm
- net VSENSE: track 35.8 -> 35.2 mm
- net TX: track 31.2 -> 31.7 mm
Other:
- board text added: "RoverWing V1.5 D. Bershadsky, A. Kirillov github.com/roverwing"
- board text removed: "POWER"
- board text removed: "RoverWing V1.2 D. Bershadsky, A. Kirillov roverwing.github.io"
