File: RoverWingBoard/Eagle/RoverWing-V1.5.sch (EAGLE design)
At the start: 82 parts, among them J1 XT30UPB-M, J10 HEADER-PH-4P, J11 HEADER-PH-3P, J12 HEADER-3X04, J13 HEADER-3X06", J14 HEADER-2X16, J15 HEADER-2X12, J16 DF13-4P-1.25DSA, J17 DF13-6P-1.25DSA, J2 HEADER-VH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

Commit message: docs update
Parts:
- C21: device RoverWing-V1.5:CAP-POL-SMD-6.3X5.4 -> RoverWing-V1.5:CAP-POL-SMD-8X10.5
Other:
- moved on the sheet: C15, C17, C18, U9
