File: RoverWingBoard/Eagle/RoverWing-V1.6.sch (EAGLE design)
At the start: 82 parts, among them J1 XT30UPB-M, J10 HEADER-PH-4P, J11 HEADER-PH-3P, J12 HEADER-3X04, J13 HEADER-3X06", J14 HEADER-2X16, J15 HEADER-2X12, J16 DF13-4P-1.25DSA, J17 DF13-6P-1.25DSA, J2 HEADER-VH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

Commit message: docs update
Parts:
- removed U7: TXS0104EPWR, RoverWing-V1.5:TXS0104EPWR
- added C16: 100nF, RoverWing-V1.5:CAP-CERAMIC-SMD0805
- added R12, R18, R19, R20: 1.8K, RoverWing-V1.5:SMD-RES-1.8K-1%-1/10W(0603)
- added R17: 1K, RoverWing-V1.5:SMD-RES-1.8K-1%-1/10W(0603)
- added R9: 1k, RoverWing-V1.5:SMD-RES-1.8K-1%-1/10W(0603)
- R10, R4: value 1k -> 1K; device RoverWing-V1.5:RES-SMD-0805 -> RoverWing-V1.5:SMD-RES-1.8K-1%-1/10W(0603)
- R11: value 1k -> 1.8K; device RoverWing-V1.5:RES-SMD-0805 -> RoverWing-V1.5:SMD-RES-1.8K-1%-1/10W(0603)
- R15, R16: value 1.8K -> 1K
Connections:
- net 3.3V: now also R12.1, R9.1; no longer R15.1, R16.1, U7.OE, U7.VCCA
- net 5V: now also C16.2; no longer U7.VCCB
- net GND: now also C16.1, R18.2, R19.2, R20.2; no longer U7.GND
- net N$10: now also R17.1; no longer U7.B2
- net N$21: now also R16.1; no longer U7.B3
- net N$7: now also R15.1; no longer U7.B4
- net SCL1: now also R11.2; no longer R13.2
- net SCL2: now also R14.2; no longer R15.2
- net SDA1: now also R12.2; no longer R14.2
- net SDA2: now also R13.2; no longer R16.2
- net SONAR1ECHO: now also R15.2, R18.1; no longer U7.A4
- net SONAR2ECHO: now also R16.2, R19.1; no longer U7.A3
- net SONAR3ECHO: now also R17.2, R20.1; no longer U7.A2
- net SWCLK: now also R9.2; no longer R11.2
Other:
- moved on the sheet: R11, R13, R14

Commit message: docs update
Parts:
- added R21: 330, RoverWing-V1.5:SMD-RES-1.8K-1%-1/10W(0603)
- renumbered U8 to U7
Connections:
- removed net NEOPIXEL_INTERNAL: D2.DI, U7A.O
- new net N$4: R21.2, U7A.O
- new net N$6: D2.DI, R21.1
Other:
- moved on the sheet: C16
Changed lines of the file:
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@@
 <part name="U$27" library="RoverWing-V1.5" deviceset="MOUNTINGHOLE" device="3.0_NPH"/>
 <part name="GND15" library="RoverWing-V1.5" deviceset="GND" device=""/>
-<part name="U8" library="RoverWing-V1.5" deviceset="74*1G125" device="DBV" technology="AHCT"/>
+<part name="U7" library="RoverWing-V1.5" deviceset="74*1G125" device="DBV" technology="AHCT"/>
 <part name="J13" library="RoverWing-V1.5" deviceset="HEADER-3X06" device="&quot;"/>
 <part name="J11" library="RoverWing-V1.5" deviceset="HEADER-PH-3P" device=""/>
@@
 <part name="R20" library="RoverWing-V1.5" deviceset="SMD-RES-1.8K-1%-1/10W(0603)" device="" value="1.8K"/>
 <part name="C16" library="RoverWing-V1.5" deviceset="CAP-CERAMIC-SMD" device="0805" value="100nF"/>
+<part name="R21" library="RoverWing-V1.5" deviceset="SMD-RES-1.8K-1%-1/10W(0603)" device="" value="330"/>
 </parts>
 <sheets>
@@
 <instance part="U$26" gate="G$1" x="35.56" y="10.16" smashed="yes"/>
 <instance part="U$27" gate="G$1" x="43.18" y="10.16" smashed="yes"/>
-<instance part="U8" gate="A" x="193.04" y="149.86" smashed="yes">
+<instance part="U7" gate="A" x="193.04" y="149.86" smashed="yes">
 <attribute name="NAME" x="185.42" y="155.575" size="1.524" layer="96" ratio="10"/>
 <attribute name="VALUE" x="171.45" y="153.67" size="1.27" layer="95" ratio="10"/>
 </instance>
-<instance part="U8" gate="P" x="198.12" y="149.86" smashed="yes"/>
+<instance part="U7" gate="P" x="198.12" y="149.86" smashed="yes"/>
 <instance part="J13" gate="G$1" x="195.58" y="88.9" smashed="yes">
 <attribute name="NAME" x="190.5" y="111.76" size="1.524" layer="96" ratio="10"/>
@@
 <attribute name="VALUE" x="117.475" y="28.8925" size="1.524" layer="96" font="vector" ratio="10"/>
 </instance>
-<instance part="D2" gate="G$1" x="220.98" y="152.4" smashed="yes"/>
+<instance part="D2" gate="G$1" x="226.06" y="152.4" smashed="yes"/>
 <instance part="GND8" gate="1" x="129.54" y="127" smashed="yes" rot="MR0">
 <attribute name="VALUE" x="132.08" y="124.46" size="1.778" layer="96" rot="MR0"/>
@@
 <attribute name="VALUE" x="41.656" y="74.168" size="1.524" layer="95" font="vector" ratio="10" rot="R270"/>
 </instance>
-<instance part="C16" gate="G$1" x="209.55" y="162.56" smashed="yes" rot="R90">
-<attribute name="NAME" x="208.28" y="158.75" size="1.524" layer="95" ratio="10" rot="R90"/>
-<attribute name="VALUE" x="212.09" y="158.75" size="1.524" layer="96" ratio="10" rot="R90"/>
+<instance part="C16" gate="G$1" x="204.47" y="162.56" smashed="yes" rot="R90">
+<attribute name="NAME" x="203.2" y="158.75" size="1.524" layer="95" ratio="10" rot="R90"/>
+<attribute name="VALUE" x="207.01" y="158.75" size="1.524" layer="96" ratio="10" rot="R90"/>
+</instance>
+<instance part="R21" gate="G$1" x="208.28" y="149.86" smashed="yes" rot="R180">
+<attribute name="NAME" x="210.82" y="148.844" size="1.524" layer="95" font="vector" ratio="10" rot="R180"/>
+<attribute name="VALUE" x="209.804" y="152.146" size="1.524" layer="95" font="vector" ratio="10" rot="R180"/>
 </instance>
 </instances>
@@
 </segment>
 <segment>
-<pinref part="U8" gate="P" pin="GND"/>
+<pinref part="U7" gate="P" pin="GND"/>
 <pinref part="D2" gate="G$1" pin="GND"/>
 <junction x="198.12" y="142.24"/>
-<wire x1="220.98" y1="142.24" x2="209.804" y2="142.24" width="0.1524" layer="91"/>
-<wire x1="209.55" y1="142.24" x2="198.12" y2="142.24" width="0.1524" layer="91"/>
+<wire x1="226.06" y1="142.24" x2="204.47" y2="142.24" width="0.1524" layer="91"/>
+<wire x1="203.2" y1="142.24" x2="198.12" y2="142.24" width="0.1524" layer="91"/>
 <wire x1="233.68" y1="144.78" x2="233.68" y2="142.24" width="0.1524" layer="91"/>
-<wire x1="233.68" y1="142.24" x2="220.98" y2="142.24" width="0.1524" layer="91"/>
-<junction x="220.98" y="142.24"/>
+<wire x1="233.68" y1="142.24" x2="226.06" y2="142.24" width="0.1524" layer="91"/>
+<junction x="226.06" y="142.24"/>
 <pinref part="J11" gate="G$1" pin="3"/>
 <wire x1="238.76" y1="144.78" x2="233.68" y2="144.78" width="0.1524" layer="91"/>
@@
 <wire x1="198.12" y1="142.24" x2="198.12" y2="137.16" width="0.1524" layer="91"/>
 <pinref part="C16" gate="G$1" pin="1"/>
-<wire x1="209.55" y1="158.75" x2="209.55" y2="142.24" width="0.1524" layer="91"/>
-<wire x1="209.55" y1="142.24" x2="209.804" y2="142.24" width="0.1524" layer="91"/>
-<junction x="209.55" y="142.24"/>
+<wire x1="204.47" y1="158.75" x2="204.47" y2="142.24" width="0.1524" layer="91"/>
+<wire x1="204.47" y1="142.24" x2="203.2" y2="142.24" width="0.1524" layer="91"/>
+<junction x="204.47" y="142.24"/>
 </segment>
 <segment>
@@
 <segment>
 <wire x1="193.04" y1="160.02" x2="193.04" y2="170.18" width="0.1524" layer="91"/>
-<pinref part="U8" gate="A" pin="OE"/>
+<pinref part="U7" gate="A" pin="OE"/>
 <pinref part="GND12" gate="1" pin="GND"/>
 </segment>
@@
 <segment>
 <pinref part="D2" gate="G$1" pin="VDD"/>
-<wire x1="226.06" y1="167.64" x2="226.06" y2="170.18" width="0.1524" layer="91"/>
-<wire x1="226.06" y1="170.18" x2="226.06" y2="175.26" width="0.1524" layer="91"/>
+<wire x1="231.14" y1="167.64" x2="231.14" y2="170.18" width="0.1524" layer="91"/>
+<wire x1="231.14" y1="170.18" x2="231.14" y2="175.26" width="0.1524" layer="91"/>
 <wire x1="236.22" y1="147.32" x2="236.22" y2="170.18" width="0.1524" layer="91"/>
-<wire x1="236.22" y1="170.18" x2="226.06" y2="170.18" width="0.1524" layer="91"/>
-<junction x="226.06" y="170.18"/>
-<pinref part="U8" gate="P" pin="VCC"/>
+<wire x1="236.22" y1="170.18" x2="231.14" y2="170.18" width="0.1524" layer="91"/>
+<junction x="231.14" y="170.18"/>
+<pinref part="U7" gate="P" pin="VCC"/>
 <wire x1="198.12" y1="157.48" x2="198.12" y2="170.18" width="0.1524" layer="91"/>
-<wire x1="198.12" y1="170.18" x2="209.55" y2="170.18" width="0.1524" layer="91"/>
-<label x="220.98" y="172.72" size="1.778" layer="95"/>
+<wire x1="198.12" y1="170.18" x2="204.47" y2="170.18" width="0.1524" layer="91"/>
+<label x="226.06" y="172.72" size="1.778" layer="95"/>
 <pinref part="J11" gate="G$1" pin="2"/>
-<wire x1="209.55" y1="170.18" x2="226.06" y2="170.18" width="0.1524" layer="91"/>
+<wire x1="204.47" y1="170.18" x2="231.14" y2="170.18" width="0.1524" layer="91"/>
 <wire x1="238.76" y1="147.32" x2="236.22" y2="147.32" width="0.1524" layer="91"/>
 <label x="236.22" y="147.32" size="1.778" layer="95"/>
 <pinref part="C16" gate="G$1" pin="2"/>
-<wire x1="209.55" y1="166.37" x2="209.55" y2="170.18" width="0.1524" layer="91"/>
-<junction x="209.55" y="170.18"/>
+<wire x1="204.47" y1="166.37" x2="204.47" y2="170.18" width="0.1524" layer="91"/>
+<junction x="204.47" y="170.18"/>
 </segment>
 </net>
@@
 <wire x1="182.88" y1="149.86" x2="180.34" y2="149.86" width="0.1524" layer="91"/>
 <label x="175.26" y="147.32" size="1.778" layer="95"/>
-<pinref part="U8" gate="A" pin="I"/>
+<pinref part="U7" gate="A" pin="I"/>
 </segment>
 </net>
@@
 <pinref part="D2" gate="G$1" pin="DO"/>
 <pinref part="J11" gate="G$1" pin="1"/>
-<wire x1="233.68" y1="149.86" x2="238.76" y2="149.86" width="0.1524" layer="91"/>
 <label x="248.92" y="152.4" size="1.778" layer="95" rot="R180"/>
-</segment>
-</net>
-<net name="NEOPIXEL_INTERNAL" class="0">
-<segment>
-<pinref part="D2" gate="G$1" pin="DI"/>
-<pinref part="U8" gate="A" pin="O"/>
-<wire x1="203.2" y1="149.86" x2="208.28" y2="149.86" width="0.1524" layer="91"/>
-<label x="205.74" y="144.78" size="1.778" layer="95" rot="R90"/>
 </segment>
 </net>
@@
 </segment>
 </net>
+<net name="N$4" class="0">
+<segment>
+<pinref part="R21" gate="G$1" pin="2"/>
+<pinref part="U7" gate="A" pin="O"/>
+<wire x1="204.47" y1="149.86" x2="203.2" y2="149.86" width="0.1524" layer="91"/>
+</segment>
+</net>
+<net name="N$6" class="0">
+<segment>
+<pinref part="R21" gate="G$1" pin="1"/>
+<pinref part="D2" gate="G$1" pin="DI"/>
+<wire x1="212.09" y1="149.86" x2="213.36" y2="149.86" width="0.1524" layer="91"/>
+</segment>
+</net>
