File: RoverWingBoard/Eagle/RoverWing-V1.6.brd (EAGLE design)
At the start: 81.3 x 81.3 mm, 82 parts, among them J1 XT30UPB-M, J10 HEADER-PH-4P, J11 HEADER-PH-3P, J12 HEADER-3X04, J13 HEADER-3X06", J14 HEADER-2X16, J15 HEADER-2X12, J16 DF13-4P-1.25DSA, J17 DF13-6P-1.25DSA, J2 HEADER-VH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

Commit message: docs update
Parts:
- removed U7: TXS0104EPWR, RoverWing-V1.5:PW14
- added C16: 100nF, RoverWing-V1.5:0805
- added R12, R18, R19, R20: 1.8K, RoverWing-V1.5:R0603
- added R17: 1K, RoverWing-V1.5:R0603
- added R9: 1k, RoverWing-V1.5:R0603
- R10, R4: value 1k -> 1K; device RoverWing-V1.5:0805 -> RoverWing-V1.5:R0603
- R11: value 1k -> 1.8K; device RoverWing-V1.5:0805 -> RoverWing-V1.5:R0603
- R15, R16: value 1.8K -> 1K
- moved R15 42.8 mm to (-0.38, -18.7)
- moved R16 42.8 mm to (2.67, -18.7)
- moved R11 34.4 mm to (-5.59, 24.3), turned to 180 degrees
- moved R13 11.3 mm to (5.71, 24.0)
- moved R14 11.1 mm to (3.17, 24.0)
- moved R10 0.40 mm to (-10.2, -28.2), turned to 90 degrees
- moved R4 0.28 mm to (-25.4, -12.2), turned to 90 degrees
Connections:
- net 3.3V: now also R12.1, R9.1; no longer R15.1, R16.1, U7.1, U7.8
- net 5V: now also C16.2; no longer U7.14
- net GND: now also C16.1, R18.2, R19.2, R20.2; no longer U7.7
- net N$10: now also R17.1; no longer U7.12
- net N$21: now also R16.1; no longer U7.11
- net N$7: now also R15.1; no longer U7.10
- net SCL1: now also R11.2; no longer R13.2
- net SCL2: now also R14.2; no longer R15.2
- net SDA1: now also R12.2; no longer R14.2
- net SDA2: now also R13.2; no longer R16.2
- net SONAR1ECHO: now also R15.2, R18.1; no longer U7.5
- net SONAR2ECHO: now also R16.2, R19.1; no longer U7.4
- net SONAR3ECHO: now also R17.2, R20.1; no longer U7.3
- net SWCLK: now also R9.2; no longer R11.2
Routing:
- net 3.3V: track 271.1 -> 260.6 mm
- net 5V: track 258.0 -> 248.0 mm, vias 19 -> 18
- net SONAR2ECHO: track 13.7 -> 18.8 mm
- net SONAR3ECHO: track 13.7 -> 18.8 mm
- net SONAR1ECHO: track 15.7 -> 19.0 mm
- net N$7: track 16.7 -> 20.0 mm
- net GND: track 43.6 -> 41.6 mm, vias 93 -> 92
- net N$10: track 28.0 -> 26.9 mm
- net N$21: track 20.7 -> 21.4 mm
- net SWCLK: track 12.4 -> 13.0 mm
Other:
- board text removed: "VCC"

Commit message: docs update
Parts:
- added R21: 330, RoverWing-V1.5:R0603
- renumbered U8 to U7
Connections:
- removed net NEOPIXEL_INTERNAL: D2.2, U7.4
- new net N$4: R21.2, U7.4
- new net N$6: D2.2, R21.1
Routing:
- net NEOPIXEL_INTERNAL: track 13.1 -> 0.00 mm
- net N$6: track 0.00 -> 7.85 mm
- net N$4: track 0.00 -> 3.51 mm

Commit message: docs update
Changed lines of the file:
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@@
 <via x="-28.956" y="4.572" extent="1-16" drill="0.35"/>
 <polygon width="0.0254" layer="1" thermals="no">
-<vertex x="-25.4" y="-6.858"/>
-<vertex x="-25.530075" y="-6.727925"/>
-<vertex x="-29.8613125" y="-6.781003125"/>
+<vertex x="-25.273" y="-6.985"/>
+<vertex x="-25.4046125" y="-6.8533875"/>
+<vertex x="-29.74246875" y="-6.906546875"/>
 <vertex x="-31.651875" y="-4.8895"/>
 <vertex x="-38.0365" y="-4.8895"/>
@@
 <vertex x="-38.989" y="-9.652"/>
 <vertex x="-25.527" y="-9.652"/>
-<vertex x="-25.4" y="-9.525"/>
+<vertex x="-25.273" y="-9.398"/>
 </polygon>
 <via x="-29.972" y="-7.62" extent="1-16" drill="0.35"/>
