File: RoverWingBoard/Eagle/RoverWing-V2.2.brd (EAGLE design)
At the start: 81.3 x 81.3 mm, 90 parts, among them J1 XT30UPB-M, J10 HEADER-3X04, J11 HEADER-3X06ANGLE, J12 HEADER-2X16, J13 HEADER-2X12, J14 DF13-4P-1.25DSA, J15 DF13-6P-1.25DSA, J16 HEADER-SH-4P, J2 HEADER-VH, J3 HEADER-VH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

Commit message: board version 2.2
Parts:
- added C22: 1uF, RoverWing-V1.5:0603
- C21: device RoverWing-V1.5:0805 -> RoverWing-V1.5:0603
- moved C21 0.25 mm to (9.65, -33.1)
Connections:
- net 5V: now also C22.2
- net GND: now also C22.1
Routing:
- net 5V: track 245.0 -> 247.2 mm
Other:
- board text added: "RoverWing V2.2 D. Bershadsky, A. Kirillov github.com/roverwing"
- board text removed: "RoverWing V2.1 D. Bershadsky, A. Kirillov github.com/roverwing"
Changed lines of the file:
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@@
 <text x="-33.9988" y="4.7888" size="1.27" layer="25" font="vector" ratio="15" rot="SR0">+</text>
 <text x="-34.3798" y="9.181196875" size="1.27" layer="25" font="vector" ratio="15" rot="SR0">-</text>
-<text x="20.574" y="13.589" size="1.27" layer="26" font="vector" ratio="11" rot="SMR270">RoverWing V2.1
+<text x="20.574" y="13.589" size="1.27" layer="26" font="vector" ratio="11" rot="SMR270">RoverWing V2.2
 D. Bershadsky, A. Kirillov
 github.com/roverwing</text>
@@
 <attribute name="NAME" x="-19.180846875" y="18.8805125" size="0.762" layer="25" font="vector" ratio="15"/>
 </element>
-<element name="C21" library="RoverWing-V1.5" package="0805" value="1uF" x="9.652" y="-32.893" smashed="yes" rot="R180">
-<attribute name="NAME" x="10.287" y="-34.163" size="0.762" layer="25" font="vector" ratio="15" rot="R180"/>
+<element name="C21" library="RoverWing-V1.5" package="0603" value="1uF" x="9.652" y="-33.147" smashed="yes" rot="R180">
+<attribute name="NAME" x="10.922" y="-34.036" size="0.762" layer="25" font="vector" ratio="15" rot="R180"/>
 </element>
 <element name="C14" library="RoverWing-V1.5" package="0603" value="100nF" x="-10.16" y="-25.654" smashed="yes" rot="R180">
@@
 <element name="D3" library="RoverWing-V1.5" package="SMA-DO214AC" package3d_urn="urn:adsk.eagle:package:43452/2" value="" x="-25.4" y="2.794" smashed="yes">
 <attribute name="MANUFACTURER" value="Comchip Technologies" x="-25.4" y="2.794" size="1.778" layer="27" display="off"/>
+<attribute name="NAME" x="-26.035" y="3.429" size="0.762" layer="25" font="vector" ratio="15"/>
 <attribute name="NAME" x="-24.13" y="2.794" size="0.5" layer="33" ratio="10" rot="R180"/>
-<attribute name="NAME" x="-26.035" y="3.429" size="0.762" layer="25" font="vector" ratio="15"/>
 <attribute name="PARTNO" value="CDBA540-HF" x="-25.4" y="2.794" size="1.778" layer="27" display="off"/>
 <attribute name="VALUE" x="-27.051" y="0" size="0.635" layer="27" ratio="10"/>
+</element>
+<element name="C22" library="RoverWing-V1.5" package="0603" value="1uF" x="4.572" y="-33.147" smashed="yes" rot="R180">
+<attribute name="NAME" x="5.715" y="-34.036" size="0.762" layer="25" font="vector" ratio="15" rot="R180"/>
+<attribute name="VALUE" x="2.967" y="-34.582" size="0.635" layer="27" ratio="10"/>
 </element>
 </elements>
@@
 <vertex x="-21.336" y="-11.684"/>
 </polygon>
+<contactref element="C22" pad="1"/>
 </signal>
 <signal name="3.3V">
@@
 <wire x1="1.8542" y1="-27.94" x2="8.052" y2="-27.94" width="0.508" layer="1"/>
 <wire x1="8.052" y1="-27.94" x2="8.052" y2="-31.928" width="0.508" layer="1"/>
-<wire x1="8.763" y1="-32.639" x2="8.763" y2="-32.893" width="0.254" layer="1"/>
+<wire x1="8.763" y1="-32.639" x2="8.89" y2="-32.893" width="0.254" layer="1"/>
 <wire x1="8.052" y1="-31.928" x2="8.763" y2="-32.639" width="0.508" layer="1"/>
 <polygon width="0.0254" layer="16" thermals="no">
@@
 <wire x1="-0.516" y1="22.217" x2="-0.508" y2="22.225" width="0.3048" layer="1"/>
 <wire x1="-4.953" y1="-11.176" x2="-3.937" y2="-11.176" width="0.254" layer="1"/>
+<wire x1="8.89" y1="-32.893" x2="8.89" y2="-33.147" width="0" layer="19" extent="1-1"/>
 </signal>
 <signal name="D+">
@@
 <wire x1="-20.447" y1="-9.271" x2="-21.463" y2="-10.287" width="0.254" layer="1"/>
 <wire x1="-21.463" y1="-10.287" x2="-27.305" y2="-10.287" width="0.254" layer="1"/>
+<contactref element="C22" pad="2"/>
+<wire x1="3.81" y1="-33.147" x2="2.286" y2="-31.623" width="0.3048" layer="1"/>
 <wire x1="3.987" y1="38.481" x2="4.064" y2="38.481" width="0" layer="19" extent="16-16"/>
 <wire x1="2.286" y1="-31.623" x2="2.286" y2="-31.75" width="0" layer="19" extent="16-16"/>

Commit message: version 2.2
Parts:
- D3: value (none) -> CDBA540-HF
Changed lines of the file:
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@@
 <attribute name="VALUE" x="-24.511" y="-6.223" size="1.27" layer="27" rot="R90"/>
 </element>
-<element name="D3" library="RoverWing-V1.5" package="SMA-DO214AC" package3d_urn="urn:adsk.eagle:package:43452/2" value="" x="-25.4" y="2.794" smashed="yes">
+<element name="D3" library="RoverWing-V1.5" package="SMA-DO214AC" package3d_urn="urn:adsk.eagle:package:43452/2" value="CDBA540-HF" x="-25.4" y="2.794" smashed="yes">
 <attribute name="MANUFACTURER" value="Comchip Technologies" x="-25.4" y="2.794" size="1.778" layer="27" display="off"/>
 <attribute name="NAME" x="-26.035" y="3.429" size="0.762" layer="25" font="vector" ratio="15"/>
