File: RoverWingBoard/Eagle/RoverWing-V2.2.brd (EAGLE design)
At the start: 81.3 x 81.3 mm, 91 parts, among them J1 XT30UPB-M, J10 HEADER-3X04, J11 HEADER-3X06ANGLE, J12 HEADER-2X16, J13 HEADER-2X12, J14 DF13-4P-1.25DSA, J15 DF13-6P-1.25DSA, J16 HEADER-SH-4P, J2 HEADER-VH, J3 HEADER-VH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

Commit message: acknowledgment of copperforge.cc  theme
Routing:
- net 3.3V: track 260.9 -> 261.4 mm
- net MOTOR1A: track 16.5 -> 17.0 mm
