File: RoverWingBoard/Eagle/RoverWing-V2.3.brd (EAGLE design)
At the start: 81.3 x 81.3 mm, 91 parts, among them J1 XT30UPB-M, J10 HEADER-3X04, J11 HEADER-3X06ANGLE, J12 HEADER-2X16, J13 HEADER-2X12, J14 DF13-4P-1.25DSA, J15 DF13-6P-1.25DSA, J16 HEADER-SH-4P, J2 HEADER-VH, J3 HEADER-VH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

Commit message: adding board design v2.3
Parts:
- moved C3 11.5 mm to (-31.9, 0.25), turned to 270 degrees
- moved R4 4.58 mm to (-31.9, -11.3), turned to 0 degrees
- moved C4 3.06 mm to (-31.9, -9.02), turned to 0 degrees
- moved U2 0.74 mm to (-28.1, -4.95)
- moved C9 0.38 mm to (-22.5, -4.32)
- moved R2 0.25 mm to (-22.5, -8.00)
Routing:
- net N$17: track 11.8 -> 4.06 mm
- net 12V: track 26.2 -> 21.6 mm
- net 5V: track 246.4 -> 250.6 mm
- net N$41: track 4.82 -> 2.28 mm
- net GND: track 32.2 -> 31.6 mm, vias 91 -> 90
- net VSENSE2: track 5.53 -> 4.90 mm
- net N$40: track 12.2 -> 11.6 mm
Other:
- board text added: "RoverWing V2.3 D. Bershadsky, A. Kirillov github.com/roverwing"
- board text removed: "RoverWing V2.2 D. Bershadsky, A. Kirillov github.com/roverwing"
